File: ulx5m-m2.kicad_sch (KiCad schematic)
At the start: 6 parts

Commit message: Initial version of 0.2
Other:
- removed sheet gpio
- sheet ethernet ports: added none; removed ID_SC, ID_SD, {DDMI1}, {ETH}, {I2C}
- sheet lvds ports: added CLKREQ#, DEVSLP, LED1#, PEDET, PERST#, PEWAKE#, SUSCLK; removed {DDMI0}
