File: ulx5m-m2.kicad_pcb (KiCad board)
At the start: 6 copper layers, 22 x 60 mm, 237 parts, among them J101 JTAG_EXT, J102 3V3_PSU, J3 Vcore_sel, J4 JTAG, J5 USB_C_Receptacle, SW1 219-2MST, U1 TLV62569DBV, U10 IS42S16320D-6BLI, U3 MPM3833CGRH-Z, U4 GateMate-CCGM1A1, U5 TLV62569DBV, U6 74LVC1G04GM,115, U7 74LVC2G00HK3-7, U8 74LVC2G00HK3-7, U9 AT25QL321-MBUE-T, X2 511FCA100M000BAG, Y1 ASE2-25.000MHZ-L-C-T

Commit message: Initial version of 0.2
Parts:
- C128, R143: moved to B.Cu
- R105, R106, R23: value 1R -> 4R7
- moved C131 6.86 mm to (62.9, 120.9)
- moved R143 6.14 mm to (58.8, 129.1), turned to 90 degrees
- moved C128 5.22 mm to (65.1, 120.1), turned to 90 degrees
- moved C132 4.78 mm to (62.0, 120.9)
- moved C54 3.03 mm to (60.5, 118.3), turned to 0 degrees
- moved C55 2.18 mm to (62.3, 118.9), turned to 180 degrees
- moved C127 2.17 mm to (65.7, 122.2), turned to 90 degrees
- moved C123 1.39 mm to (66.8, 124.8), turned to 90 degrees
- moved C125 1.36 mm to (65.8, 124.8), turned to 90 degrees
- moved C53 1.34 mm to (60.1, 117.4), turned to 0 degrees
- moved TP8 1.11 mm to (64.0, 121.6)
- moved C138 0.57 mm to (62.4, 128.2)
- moved C56 0.05 mm to (66.7, 122.1)
- moved R7 0.05 mm to (63.7, 123.8)
- turned R105 to 180 degrees
Connections:
- net /lvds/+1V2_SA renamed /lvds/+3V3_SA
- C120 pad 1: VDD_CORE -> VDD_SER_PLL
- C121 pad 1: VDD_CORE -> VDD_SER
- C122 pad 1: VDD_CORE -> VDD_SER_PLL
- C123 pad 1: VDD_CORE -> VDD_SER
- C124 pad 1: VDD_CORE -> VDD_SER_PLL
- C125 pad 1: VDD_CORE -> VDD_SER
- C127 pad 1: VDD_SER_PLL -> VDD_CORE
- C128 pad 1: VDD_SER -> VDD_CORE
- C33 pad 1: VDD_CORE -> VDD_PLL
- C36 pad 1: VDD_CORE -> VDD_PLL
- C39 pad 1: VDD_CORE -> VDD_PLL
- C42 pad 1: VDD_PLL -> VDD_CORE
- C49 pad 1: +1V2 -> +3V3
- R121 pad 1: +1V2 -> +3V3
- U4 pad M17: /lvds/PEDET -> unconnected-(U4E-IO_SB_A3-PadM17)
- U4 pad M18: /lvds/LED1# -> unconnected-(U4E-IO_SB_B3-PadM18)
- U4 pad P17: /lvds/PEWAKE# -> unconnected-(U4E-IO_SB_A2-PadP17)
- U4 pad P18: /lvds/SUSCLK -> unconnected-(U4E-IO_SB_B2-PadP18)
- U4 pad R10: /lvds/LVDS0_D1_P -> unconnected-(U4E-IO_SA_A7-PadR10)
- U4 pad R17: /lvds/PERST# -> unconnected-(U4E-IO_SB_A1-PadR17)
- U4 pad R18: /lvds/CLKREQ# -> unconnected-(U4E-IO_SB_B1-PadR18)
- U4 pad R6: /lvds/LVDS1_C_P -> /PERST#
- U4 pad R7: /lvds/LVDS1_D1_P -> /DEVSLP
- U4 pad R8: /lvds/LVDS0_D3_P -> unconnected-(U4E-IO_SA_A4-PadR8)
- U4 pad R9: /lvds/LVDS0_C_P -> unconnected-(U4E-IO_SA_A6-PadR9)
- U4 pad T10: /lvds/LVDS0_D1_N -> unconnected-(U4E-IO_SA_B7-PadT10)
- U4 pad T6: /lvds/LVDS1_C_N -> /LED1#
- U4 pad T7: /lvds/LVDS1_D1_N -> /SUSCLK
- U4 pad T8: /lvds/LVDS0_D3_N -> unconnected-(U4E-IO_SA_B4-PadT8)
- U4 pad T9: /lvds/LVDS0_C_N -> unconnected-(U4E-IO_SA_B6-PadT9)
- U4 pad U10: /lvds/LVDS0_D0_P -> unconnected-(U4E-IO_SA_A8-PadU10)
- U4 pad U18: /lvds/DEVSLP -> unconnected-(U4E-IO_SB_B0-PadU18)
- U4 pad U5: /lvds/LVDS1_D2_P -> unconnected-(U4E-IO_SA_A0-PadU5)
- U4 pad U7: /lvds/LVDS1_D0_P -> /PEWAKE#
- U4 pad U8: /lvds/LVDS0_D2_P -> unconnected-(U4E-IO_SA_A5-PadU8)
- U4 pad V10: /lvds/LVDS0_D0_N -> unconnected-(U4E-IO_SA_B8-PadV10)
- U4 pad V5: /lvds/LVDS1_D2_N -> /PEDET
- U4 pad V7: /lvds/LVDS1_D0_N -> /CLKREQ#
- U4 pad V8: /lvds/LVDS0_D2_N -> unconnected-(U4E-IO_SA_B5-PadV8)
Routing:
- net +3V3: track 268.6 -> 291.8 mm
- net /LED1#: track 2.93 -> 22.0 mm, vias 1 -> 2
- net VDD_CORE: track 295.2 -> 276.4 mm, vias 35 -> 32
- net /SUSCLK: track 0.17 -> 17.7 mm, vias 0 -> 1
- net /PERST#: track 0.00 -> 16.6 mm, vias 0 -> 2
- net /PEWAKE#: track 0.00 -> 15.3 mm, vias 0 -> 1
- net /CLKREQ#: track 0.00 -> 14.3 mm, vias 0 -> 1
- net /PEDET: track 0.00 -> 13.7 mm
- net /DEVSLP: track 3.01 -> 15.8 mm, vias 0 -> 2
- net /config/~{CFG_FAIL}: track 14.8 -> 24.0 mm
- net VDD_SER_PLL: track 5.17 -> 13.9 mm, vias 2 -> 1
- net GND: track 810.4 -> 818.2 mm
- net /config/CFG_DONE: track 13.9 -> 19.9 mm
- net VDD_CLK: track 129.0 -> 134.8 mm, vias 23 -> 24
- net /lvds/+1V8_SB: track 44.6 -> 41.0 mm
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- added copper zone on In3.Cu, net GND
- added copper zone on In4.Cu, net GND
- removed copper zone on In2.Cu, net GND

Commit message: Update stackup
Parts:
- R105, R106, R23: value 4R7 -> 2R
- moved R110 0.38 mm to (60.6, 124.4)
Routing:
- net /PEWAKE#: track 15.3 -> 16.7 mm
- net /CLKREQ#: track 14.3 -> 15.1 mm
- net /config/CFG_DONE: track 19.9 -> 19.2 mm
Other:
- board text added: "JLC06081H-1080"
- board text removed: "JLC06081H-7628"
