File: ulx5m-m2.kicad_pcb (KiCad board)
At the start: 6 copper layers, 22 x 60 mm, 237 parts, among them J101 JTAG_EXT, J102 3V3_PSU, J3 Vcore_sel, J4 JTAG, J5 USB_C_Receptacle, SW1 219-2MST, U1 TLV62569DBV, U10 IS42S16320D-6BLI, U3 MPM3833CGRH-Z, U4 GateMate-CCGM1A1, U5 TLV62569DBV, U6 74LVC1G04GM,115, U7 74LVC2G00HK3-7, U8 74LVC2G00HK3-7, U9 AT25QL321-MBUE-T, X2 511FCA100M000BAG, Y1 ASE2-25.000MHZ-L-C-T

Commit message: Before adding teardrops
Routing:
- net GND: vias 197 -> 222
Changed lines of the file:
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@@
+	)
+	(via
+		(at 57.89 81.52)
+		(size 0.45)
+		(drill 0.2)
+		(layers "F.Cu" "B.Cu")
+		(free yes)
+		(net "GND")
 	)
 	(via
@@
 	)
 	(via
+		(at 48.52 88.09)
+		(size 0.45)
+		(drill 0.2)
+		(layers "F.Cu" "B.Cu")
+		(free yes)
+		(net "GND")
+	)
+	(via
 		(at 54.03 91.72)
 		(size 0.45)
@@
 		)
 		(filling no)
+		(net "GND")
+	)
+	(via
+		(at 50.28 89.35)
+		(size 0.45)
+		(drill 0.2)
+		(layers "F.Cu" "B.Cu")
+		(free yes)
+		(net "GND")
+	)
+	(via
+		(at 52.16 98.57)
+		(size 0.45)
+		(drill 0.2)
+		(layers "F.Cu" "B.Cu")
+		(free yes)
 		(net "GND")
 	)
@@
 	)
 	(via
+		(at 48.42 93.57)
+		(size 0.45)
+		(drill 0.2)
+		(layers "F.Cu" "B.Cu")
+		(free yes)
+		(net "GND")
+	)
+	(via
 		(at 59.38 93.17)
 		(size 0.45)
@@
 	)
 	(via
+		(at 59.62 86.67)
+		(size 0.45)
+		(drill 0.2)
+		(layers "F.Cu" "B.Cu")
+		(free yes)
+		(net "GND")
+	)
+	(via
 		(at 59.61 81.32)
 		(size 0.45)
@@
 		)
 		(filling no)
+		(net "GND")
+	)
+	(via
+		(at 51.64 102.51)
+		(size 0.45)
+		(drill 0.2)
+		(layers "F.Cu" "B.Cu")
+		(free yes)
 		(net "GND")
 	)
@@
 	)
 	(via
+		(at 48.43 102.93)
+		(size 0.45)
+		(drill 0.2)
+		(layers "F.Cu" "B.Cu")
+		(free yes)
+		(net "GND")
+	)
+	(via
 		(at 60.27 128.02)
 		(size 0.45)
@@
 		(drill 0.2)
 		(layers "F.Cu" "B.Cu")
+		(net "GND")
+	)
+	(via
+		(at 65.21 86.57)
+		(size 0.45)
+		(drill 0.2)
+		(layers "F.Cu" "B.Cu")
+		(free yes)
 		(net "GND")
 	)
@@
 	)
 	(via
+		(at 48.43 98.88)
+		(size 0.45)
+		(drill 0.2)
+		(layers "F.Cu" "B.Cu")
+		(free yes)
+		(net "GND")
+	)
+	(via
 		(at 60.959999 117.49)
 		(size 0.4)
@@
 	)
 	(via
+		(at 48.43 94.9)
+		(size 0.45)
+		(drill 0.2)
+		(layers "F.Cu" "B.Cu")
+		(free yes)
+		(net "GND")
+	)
+	(via
 		(at 51.72 93.16)
 		(size 0.45)
@@
 	)
 	(via
+		(at 62.86 84.44)
+		(size 0.45)
+		(drill 0.2)
+		(layers "F.Cu" "B.Cu")
+		(free yes)
+		(net "GND")
+	)
+	(via
 		(at 65.38 106.99)
 		(size 0.4)
@@
 		)
 		(filling no)
+		(net "GND")
+	)
+	(via
+		(at 50.39 92.39)
+		(size 0.45)
+		(drill 0.2)
+		(layers "F.Cu" "B.Cu")
+		(free yes)
 		(net "GND")
 	)
@@
 	)
 	(via
+		(at 67.87 79.33)
+		(size 0.45)
+		(drill 0.2)
+		(layers "F.Cu" "B.Cu")
+		(free yes)
+		(net "GND")
+	)
+	(via
 		(at 55.03 104.83)
 		(size 0.45)
@@
 		)
 		(filling no)
+		(net "GND")
+	)
+	(via
+		(at 50.51 109.2)
+		(size 0.45)
+		(drill 0.2)
+		(layers "F.Cu" "B.Cu")
+		(free yes)
 		(net "GND")
 	)
@@
 	)
 	(via
+		(at 52.14 97.82)
+		(size 0.45)
+		(drill 0.2)
+		(layers "F.Cu" "B.Cu")
+		(free yes)
+		(net "GND")
+	)
+	(via
 		(at 65.14 124.83)
 		(size 0.45)
@@
 	)
 	(via
+		(at 61.24 95.16)
+		(size 0.45)
+		(drill 0.2)
+		(layers "F.Cu" "B.Cu")
+		(free yes)
+		(net "GND")
+	)
+	(via
 		(at 63.62 128)
 		(size 0.45)
@@
 	)
 	(via
+		(at 56.95 94.63)
+		(size 0.45)
+		(drill 0.2)
+		(layers "F.Cu" "B.Cu")
+		(free yes)
+		(net "GND")
+	)
+	(via
 		(at 55.389999 112.64)
 		(size 0.4)
@@
 	)
 	(via
+		(at 60.29 94.13)
+		(size 0.45)
+		(drill 0.2)
+		(layers "F.Cu" "B.Cu")
+		(free yes)
+		(net "GND")
+	)
+	(via
 		(at 65.76 110.56)
 		(size 0.4)
@@
 	)
 	(via
+		(at 60.24 79.1)
+		(size 0.45)
+		(drill 0.2)
+		(layers "F.Cu" "B.Cu")
+		(free yes)
+		(net "GND")
+	)
+	(via
 		(at 65.61 131.1)
 		(size 0.4)
@@
 		)
 		(filling no)
+		(net "GND")
+	)
+	(via
+		(at 51.4 106.68)
+		(size 0.45)
+		(drill 0.2)
+		(layers "F.Cu" "B.Cu")
+		(free yes)
 		(net "GND")
 	)
@@
 	)
 	(via
+		(at 68.07 83.72)
+		(size 0.45)
+		(drill 0.2)
+		(layers "F.Cu" "B.Cu")
+		(free yes)
+		(net "GND")
+	)
+	(via
 		(at 58.589999 111.840001)
 		(size 0.4)
@@
 		(drill 0.2)
 		(layers "F.Cu" "B.Cu")
+		(net "GND")
+	)
+	(via
+		(at 52.67 92.85)
+		(size 0.45)
+		(drill 0.2)
+		(layers "F.Cu" "B.Cu")
+		(free yes)
 		(net "GND")
 	)
@@
 	)
 	(via
+		(at 52.08 97.04)
+		(size 0.45)
+		(drill 0.2)
+		(layers "F.Cu" "B.Cu")
+		(free yes)
+		(net "GND")
+	)
+	(via
 		(at 55.39 111.04)
 		(size 0.4)
@@
 		(net "GND")
 	)
+	(via
+		(at 54.18 81.83)
+		(size 0.45)
+		(drill 0.2)
+		(layers "F.Cu" "B.Cu")
+		(free yes)
+		(net "GND")
+	)

Commit message: Changing footprint - adding teardrops
Parts:
- removed R107, R108, R110: dnp, Resistor_SMD:R_0402_1005Metric
- C136, C137, C143, C144, C145, C146, C147, C148, C149, C150: footprint Capacitor_SMD:C_0402_1005Metric -> Capacitors_impedance:C_0402_SI_M
Routing:
- net GND: track 818.2 -> 815.8 mm
- removed copper zone on B.Cu, net GND
- removed copper zone on F.Cu, net GND
