File: config.kicad_sch (KiCad schematic)
At the start: 43 parts, among them J101 JTAG_EXT, J102 3V3_PSU, J4 JTAG, SW1 219-2MST, U4 GateMate-CCGM1A1, U6 74LVC1G04GM,115, U7 74LVC2G00HK3-7, U8 74LVC2G00HK3-7, U9 AT25QL321-MBUE-T

Commit message: initial version of ULX5-PCIe-1x
Parts:
- R147, R148, R149, R150: value 10k -> 27R; now fitted; now in the parts list
Connections:
- net GND: now also SW1.5
- net PI_TMS: now reaches J101.4 (Pin_4), J4.4 (Pin_4), R43.2
- net PI_TCK: now reaches J101.1 (Pin_1), J4.1 (Pin_1), R40.2
- net PI_TDI: now reaches J101.2 (Pin_2), J4.2 (Pin_2), R41.2
- net PI_TDO: now reaches J101.3 (Pin_3), J4.3 (Pin_3), R42.2
- net GPIO12 renamed TDI
- net GPIO16 renamed TDO
- net GPIO20 renamed TCK
- net GPIO21 renamed TMS
- no-connect marks 0 -> 2
Other:
- moved on the sheet: J101
