File: ethernet.kicad_sch (KiCad schematic)
At the start: 50 parts, among them J5 USB_C_Receptacle, U4 GateMate-CCGM1A1

Commit message: initial version of ULX5-PCIe-1x
Connections:
- net VDD_CLK is gone; now on net +3V3: R144.1, R145.1, R146.1
