File: decap.kicad_sch (KiCad schematic)
At the start: 2 parts

Commit message: Adding 12V PSU
Other:
- company: (none) -> ${project_creator}
- title: (none) -> ${project_name}
Changed lines of the file:
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@@
 	(generator_version "10.0")
 	(paper "A4")
+	(title_block
+		(title "${project_name}")
+		(date "2025-06-24")
+		(rev "${project_version}")
+		(company "${project_creator}")
+		(comment 1 "${project_license}")
+	)
 	(wire
 		(pts
