File: ulx5-PCIe-1x.kicad_pcb (KiCad board)
At the start: 6 copper layers, 167.7 x 68.9 mm, 261 parts, among them J1 PCIexpress_bracket, J101 JTAG_EXT, J102 3V3_PSU, J2 PCIexpress_x1, J3 Vcore_sel, J303 Conn_01x22_Female, J4 JTAG, J5 USB_C_Receptacle, SW1 219-2MST, U1 TLV62569DBV, U10 IS42S16320D-6BLI, U3 MPM3833CGRH-Z, U4 GateMate-CCGM1A1, U5 TLV62569DBV, U6 74LVC1G04GM,115, U7 74LVC2G00HK3-7, U8 74LVC2G00HK3-7, U9 AT25QL321-MBUE-T, X2 511FCA100M000BAG, Y1 ASE2-25.000MHZ-L-C-T

Commit message: power enable fix - connecting AGND
Parts:
- R2: value 51k -> 100k
Connections:
- A101 pad 33: unconnected-(A101-AGND-Pad33) -> GND
Routing:
- net GND: track 845.6 -> 847.3 mm, vias 261 -> 262
- added copper zone on In3.Cu, net GND
- added copper zone on In4.Cu, net GND
Changed lines of the file:
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@@
 			)
 		)
-		(attr smd)
+		(attr smd dnp)
 		(duplicate_pad_numbers_are_jumpers no)
 		(fp_line
@@
 			(size 1.6 0.8)
 			(layers "F.Cu" "F.Mask")
-			(net "unconnected-(A101-AGND-Pad33)")
+			(net "GND")
 			(pinfunction "AGND_33")
 			(pintype "power_out")
@@
 			)
 		)
-		(attr smd)
+		(attr smd dnp)
 		(duplicate_pad_numbers_are_jumpers no)
 		(fp_line
@@
 			(remove_unused_layers yes)
 			(keep_end_layers yes)
-			(zone_layer_connections "In1.Cu" "In2.Cu")
+			(zone_layer_connections "In1.Cu" "In2.Cu" "In3.Cu" "In4.Cu")
 			(net "GND")
 			(pinfunction "SHIELD_S")
@@
 			)
 		)
-		(property "Value" "51k"
+		(property "Value" "100k"
 			(at 0 -1.17 0)
 			(layer "B.Fab")
@@
 			)
 		)
-		(property "LCSC" "C144749"
+		(property "LCSC" ""
 			(at 0 0 180)
 			(unlocked yes)
@@
 	)
 	(segment
+		(start 190.00474 202.78026)
+		(end 190.00474 204.44026)
+		(width 0.5)
+		(layer "F.Cu")
+		(net "GND")
+	)
+	(segment
 		(start 127.067082 216.459512)
 		(end 127.467083 216.059512)
@@
 	)
 	(segment
+		(start 190.00474 204.44026)
+		(end 190.05474 204.49026)
+		(width 0.5)
+		(layer "F.Cu")
+		(net "GND")
+	)
+	(segment
 		(start 127.147082 223.739513)
 		(end 127.067082 223.659513)
@@
 	)
 	(via
+		(at 190.05474 204.49026)
+		(size 0.45)
+		(drill 0.2)
+		(layers "F.Cu" "B.Cu")
+		(net "GND")
+	)
+	(via
 		(at 202.68474 181.67026)
 		(size 0.45)
@@
 	)
 	(segment
+		(start 79.474741 221.352759)
+		(end 79.01724 221.81026)
+		(width 0.5)
+		(layer "F.Cu")
+		(net "Net-(LED_P501-Pad2)")
+	)
+	(segment
+		(start 79.474741 220.580259)
+		(end 79.474741 221.352759)
+		(width 0.5)
+		(layer "F.Cu")
+		(net "Net-(LED_P501-Pad2)")
+	)
+	(segment
+		(start 79.75474 220.30026)
+		(end 79.474741 220.580259)
+		(width 0.5)
+		(layer "F.Cu")
+		(net "Net-(LED_P501-Pad2)")
+	)
+	(segment
 		(start 88.399739 216.010259)
 		(end 88.399739 216.99526)
@@
 		(net "Net-(J3-Pin_1)")
 	)
-	(segment
-		(start 79.474741 221.352759)
-		(end 79.01724 221.81026)
-		(width 0.5)
-		(layer "F.Cu")
-		(net "Net-(LED_P501-Pad2)")
-	)
-	(segment
-		(start 79.474741 220.580259)
-		(end 79.474741 221.352759)
-		(width 0.5)
-		(layer "F.Cu")
-		(net "Net-(LED_P501-Pad2)")
-	)
-	(segment
-		(start 79.75474 220.30026)
-		(end 79.474741 220.580259)
-		(width 0.5)
-		(layer "F.Cu")
-		(net "Net-(LED_P501-Pad2)")
-	)
 	(zone
 		(net "VDD_SER")
@@
 		(layer "F.Cu")
 		(hatch none 0.1)
-		(priority 30077)
+		(priority 30076)
 		(attr
 			(teardrop
@@
 		(layer "F.Cu")
 		(hatch none 0.1)
-		(priority 30076)
+		(priority 30077)
 		(attr
 			(teardrop
@@
 		(layer "F.Cu")
 		(hatch none 0.1)
-		(priority 30067)
+		(priority 30068)
 		(attr
 			(teardrop
@@
 		(layer "F.Cu")
 		(hatch none 0.1)
-		(priority 30068)
+		(priority 30067)
 		(attr
 			(teardrop
@@
 		(layer "F.Cu")
 		(hatch none 0.1)
-		(priority 30072)
+		(priority 30071)
 		(attr
 			(teardrop
@@
 		(layer "F.Cu")
 		(hatch none 0.1)
-		(priority 30071)
+		(priority 30072)
 		(attr
 			(teardrop
@@
 		(net "GND")
 		(layer "In1.Cu")
-		(hatch edge 0.508)
-		(connect_pads thru_hole_only
-			(clearance 0)
-		)
-		(min_thickness 0.25)
-		(fill yes
-			(thermal_gap 0.508)
-			(thermal_bridge_width 0.508)
-			(island_removal_mode 0)
-		)
-		(polygon
-			(pts
-				(xy 43.65474 176.26526) (xy 211.27974 176.26526) (xy 211.27974 232.39026) (xy 109.02974 232.39026)
-				(xy 109.02974 239.54026) (xy 88.52974 239.54026) (xy 88.52974 234.26526) (xy 85.02974 234.26526)
-				(xy 85.02974 237.01526) (xy 76.90474 237.01526) (xy 76.90474 232.39026) (xy 58.65474 232.39026)
-				(xy 58.65474 240.64026) (xy 43.65474 240.64026)
-			)
-		)
-	)
-	(zone
-		(net "GND")
-		(layer "In1.Cu")
 		(hatch none 0.1)
 		(priority 30014)
@@
 	)
 	(zone
+		(net "GND")
+		(layers "In1.Cu" "In2.Cu" "In3.Cu" "In4.Cu")
+		(hatch edge 0.508)
+		(connect_pads thru_hole_only
+			(clearance 0)
+		)
+		(min_thickness 0.25)
+		(fill yes
+			(thermal_gap 0.508)
+			(thermal_bridge_width 0.508)
+			(island_removal_mode 0)
+		)
+		(polygon
+			(pts
+				(xy 43.65474 176.26526) (xy 211.27974 176.26526) (xy 211.27974 232.39026) (xy 109.02974 232.39026)
+				(xy 109.02974 239.54026) (xy 88.52974 239.54026) (xy 88.52974 234.26526) (xy 85.02974 234.26526)
+				(xy 85.02974 237.01526) (xy 76.90474 237.01526) (xy 76.90474 232.39026) (xy 58.65474 232.39026)
+				(xy 58.65474 240.64026) (xy 43.65474 240.64026)
+			)
+		)
+	)
+	(zone
 		(net "RST_N")
 		(layer "In2.Cu")
@@
 			)
 		)
-	)
-	(zone
-		(net "GND")
-		(layer "In2.Cu")
-		(hatch edge 0.508)
-		(connect_pads thru_hole_only
-			(clearance 0)
-		)
-		(min_thickness 0.25)
-		(fill yes
-			(thermal_gap 0.508)
-			(thermal_bridge_width 0.508)
-			(island_removal_mode 0)
-		)
-		(polygon
-			(pts
-				(xy 43.65474 176.26526) (xy 211.27974 176.26526) (xy 211.27974 232.39026) (xy 109.02974 232.39026)
-				(xy 109.02974 239.54026) (xy 88.52974 239.54026) (xy 88.52974 234.26526) (xy 85.02974 234.26526)
-				(xy 85.02974 237.01526) (xy 76.90474 237.01526) (xy 76.90474 232.39026) (xy 58.65474 232.39026)
-				(xy 58.65474 240.64026) (xy 43.65474 240.64026)
-			)
-		)
