File: ulx5-PCIe-1x.kicad_pcb (KiCad board)
At the start: 6 copper layers, 167.7 x 68.9 mm, 261 parts, among them J1 PCIexpress_bracket, J101 JTAG_EXT, J102 3V3_PSU, J2 PCIexpress_x1, J3 Vcore_sel, J303 Conn_01x22_Female, J4 JTAG, J5 USB_C_Receptacle, SW1 219-2MST, U1 TLV62569DBV, U10 IS42S16320D-6BLI, U3 MPM3833CGRH-Z, U4 GateMate-CCGM1A1, U5 TLV62569DBV, U6 74LVC1G04GM,115, U7 74LVC2G00HK3-7, U8 74LVC2G00HK3-7, U9 AT25QL321-MBUE-T, X2 511FCA100M000BAG, Y1 ASE2-25.000MHZ-L-C-T

Commit message: Fixing diff lines
Parts:
- removed D101: D_Shockley, Diode_SMD:D_SMA
- added D301: D_Schottky, Diode_SMD:D_SMA, F.Cu at (196.1, 209.7)
- added JP303: LVDS-1V2-1V8, Jumper:SolderJumper-3_P1.3mm_Bridged2Bar12_RoundedPad1.0x1.5mm, F.Cu at (110.0, 208.3)
- added LED_P502: LowCur_green, LED_SMD:LED_0603_1608Metric, F.Cu at (109.0, 229.6)
- added R508: 560R 1%, Resistor_SMD:R_0402_1005Metric, F.Cu at (108.5, 228.3)
- U10: value IS42S16320D-6BLI -> IS42VM16320E
- moved SW1 2.92 mm to (108.3, 203.6)
- moved TP11 1.07 mm to (123.6, 226.4)
- moved C138 0.40 mm to (111.9, 221.1)
- moved R111 0.39 mm to (112.0, 222.1)
Connections:
- C49 pad 1: +1V2 -> Net-(JP303-C)
- J2 pad B12: unconnected-(J2-RSVD-PadB12) -> /CLKREQ#
- R121 pad 1: +1V2 -> Net-(JP303-C)
- U4 pad R18: /LED1# -> /lvds/LED1#
Routing:
- net /CLKREQ#: track 0.80 -> 33.3 mm, vias 0 -> 2
- net /lvds/LED1#: track 0.00 -> 19.4 mm, vias 0 -> 2
- net Net-(JP303-C): track 0.00 -> 9.08 mm, vias 0 -> 1
- net VDD_CLK: track 190.0 -> 195.3 mm, vias 19 -> 20
- net /config/JTAG_CFG_MD3: track 15.5 -> 20.4 mm
- net Net-(LED_P502-Pad2): track 0.00 -> 1.68 mm
- net /config/JTAG_CFG_MD2: track 15.7 -> 17.1 mm
- net +1V2: track 14.0 -> 12.9 mm, vias 0 -> 1
- net GND: track 847.3 -> 848.2 mm, vias 262 -> 263
- net /LED1#: track 0.75 -> 0.00 mm
- net /serdes/SER_CK_P: track 9.06 -> 8.43 mm
