File: ulx5-PCIe-1x.kicad_pcb (KiCad board)
At the start: 6 copper layers, 167.7 x 68.9 mm, 264 parts, among them J1 PCIexpress_bracket, J101 JTAG_EXT, J102 3V3_PSU, J2 PCIexpress_x1, J3 Vcore_sel, J303 Conn_01x22_Female, J4 JTAG, J5 USB_C_Receptacle, SW1 219-2MST, U1 TLV62569DBV, U10 IS42VM16320E, U3 MPM3833CGRH-Z, U4 GateMate-CCGM1A1, U5 TLV62569DBV, U6 74LVC1G04GM,115, U7 74LVC2G00HK3-7, U8 74LVC2G00HK3-7, U9 AT25QL321-MBUE-T, X2 511FCA100M000BAG, Y1 ASE2-25.000MHZ-L-C-T

Commit message: Adding stackup
Other:
- board text removed: "JLC06081H-1080"
- board text removed: "Napajanje!! 12V"
