File: ram.kicad_sch (KiCad schematic)
At the start: 25 parts, among them U10 IS42S16320D-6BLI, U4 GateMate-CCGM1A1

Commit message: initial version of ULX5-PCIe-1x
Connections:
- net +3V3: now also C57.1, C58.1, C75.1, C76.1, U4.H5 (VDD_WB), U4.J2 (VDD_WB), U4.K5 (VDD_WB), U4.M2 (VDD_WB), U4.M5 (VDD_WB); no longer C101.1, C140.1, C141.1, C85.1, C99.1
- net SDRAM_VCC: now also C101.1, C140.1, C141.1, C85.1, C99.1; no longer C57.1, C58.1, C75.1, C76.1, U4.H5 (VDD_WB), U4.J2 (VDD_WB), U4.K5 (VDD_WB), U4.M2 (VDD_WB), U4.M5 (VDD_WB)
- net FPGA_UART_TX: now reaches U4.H1 (IO_WB_A7)
- net FPGA_UART_RX: now reaches U4.H2 (IO_WB_B7)
- net FPGA_GPIO1: now reaches U4.H3 (IO_WB_A8)
- net FPGA_GPIO2: now reaches U4.H4 (IO_WB_B8)
- net SCL0: now reaches U4.M3 (IO_WB_A1)
- net SDA0: now reaches U4.M4 (IO_WB_B1)
- net CAM_GPIO0: now reaches U4.N1 (IO_WB_A0)
- net CAM_GPIO1: now reaches U4.N2 (IO_WB_B0)

Commit message: update
Parts:
- U10: value IS42S16320D-6BLI -> IS42VM16320E
Other:
- moved on the sheet: C86, C87, C88, C89, C90, C91, C92, C93, R115, R116, U4C
