File: PCIexpress_connector.kicad_sch (KiCad schematic)
At the start: 1 part, among them J2 PCIexpress_x1

Commit message: Adding 12V PSU
Parts:
- added JP302: Jumper_2_Bridged, Jumper:SolderJumper-2_P1.3mm_Bridged2Bar_RoundedPad1.0x1.5mm, symbol Jumper:Jumper_2_Bridged
Connections:
- net +3V3: now also JP302.1 (A); no longer J2.A10 (+3.3V), J2.A9 (+3.3V), J2.B8 (+3.3V)
- new net +3V3_PCIe: J2.A10 (+3.3V), J2.A9 (+3.3V), J2.B8 (+3.3V), JP302.2 (B)
Changed lines of the file:
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@@
+	)
+	(symbol
+		(lib_id "Jumper:Jumper_2_Bridged")
+		(at 66.04 68.58 0)
+		(unit 1)
+		(body_style 1)
+		(exclude_from_sim no)
+		(in_bom yes)
+		(on_board yes)
+		(in_pos_files yes)
+		(dnp no)
+		(fields_autoplaced yes)
+		(property "Reference" "JP302"
+			(at 66.04 63.5 0)
+			(show_name no)
+			(do_not_autoplace no)
+			(effects
+				(font
+					(size 1.27 1.27)
+				)
+			)
+		)
+		(property "Value" "Jumper_2_Bridged"
+			(at 66.04 66.04 0)
+			(show_name no)
+			(do_not_autoplace no)
+			(effects
+				(font
+					(size 1.27 1.27)
+				)
+			)
+		)
+		(property "Footprint" "Jumper:SolderJumper-2_P1.3mm_Bridged2Bar_RoundedPad1.0x1.5mm"
+			(at 66.04 68.58 0)
+			(hide yes)
+			(show_name no)
+			(do_not_autoplace no)
+			(effects
+				(font
+					(size 1.27 1.27)
+				)
+			)
+		)
+		(property "Datasheet" ""
+			(at 66.04 73.66 0)
+			(hide yes)
+			(show_name no)
+			(do_not_autoplace no)
+			(effects
+				(font
+					(size 1.27 1.27)
+				)
+			)
+		)
+		(property "Description" "Jumper, 2-pole, closed/bridged"
+			(at 66.04 76.2 0)
+			(hide yes)
+			(show_name no)
+			(do_not_autoplace no)
+			(effects
+				(font
+					(size 1.27 1.27)
+				)
+			)
+		)
+		(pin "2"
+		)
+		(pin "1"
+		)
+		(instances
+			(project "ulx5-PCIe-1x"
+				(path "/9e5cbfd6-8186-4817-919e-acd256336bc8/3b67bf4d-c966-4618-b78c-abe52a948139"
+					(reference "JP302")
+					(unit 1)
+				)
+			)
+		)
 	)
 	(symbol
@@
 	(symbol
 		(lib_id "PCIexpress_x1_low-rescue:+3.3V-power")
+		(at 60.96 68.58 90)
+		(unit 1)
+		(body_style 1)
+		(exclude_from_sim no)
+		(in_bom yes)
+		(on_board yes)
+		(in_pos_files yes)
+		(dnp no)
+		(property "Reference" "#PWR0181"
+			(at 64.77 68.58 0)
+			(hide yes)
+			(show_name no)
+			(do_not_autoplace no)
+			(effects
+				(font
+					(size 1.27 1.27)
+				)
+			)
+		)
+		(property "Value" "+3V3"
+			(at 57.7088 68.199 90)
+			(show_name no)
+			(do_not_autoplace no)
+			(effects
+				(font
+					(size 1.27 1.27)
+				)
+				(justify left)
+			)
+		)
+		(property "Footprint" ""
+			(at 60.96 68.58 0)
+			(hide yes)
+			(show_name no)
+			(do_not_autoplace no)
+			(effects
+				(font
+					(size 1.27 1.27)
+				)
+			)
+		)
+		(property "Datasheet" ""
+			(at 60.96 68.58 0)
+			(hide yes)
+			(show_name no)
+			(do_not_autoplace no)
+			(effects
+				(font
+					(size 1.27 1.27)
+				)
+			)
+		)
+		(property "Description" ""
+			(at 60.96 68.58 0)
+			(show_name no)
+			(do_not_autoplace no)
+			(effects
+				(font
+					(size 1.27 1.27)
+				)
+			)
+		)
+		(pin "1"
+		)
+		(instances
+			(project "ulx5-PCIe-1x"
+				(path "/9e5cbfd6-8186-4817-919e-acd256336bc8/3b67bf4d-c966-4618-b78c-abe52a948139"
+					(reference "#PWR0181")
+					(unit 1)
+				)
+			)
+		)
+	)
+	(symbol
+		(lib_id "PCIexpress_x1_low-rescue:+3.3V-power")
 		(at 161.29 71.12 270)
 		(unit 1)
@@
 			)
 		)
-		(property "Value" "+3V3"
+		(property "Value" "+3V3_PCIe"
 			(at 164.5412 71.501 90)
 			(show_name no)
@@
 			)
 		)
-		(property "Value" "+3V3"
+		(property "Value" "+3V3_PCIe"
 			(at 117.3988 68.199 90)
 			(show_name no)
@@
 			)
 		)
-		(property "Value" "+3V3"
+		(property "Value" "+3V3_PCIe"
 			(at 164.5412 74.041 90)
 			(show_name no)
@@
 					(unit 1)
 				)
+			)
+		)
+	)
+	(symbol
+		(lib_id "PCIexpress_x1_low-rescue:+3.3V-power")
+		(at 71.12 68.58 270)
+		(unit 1)
+		(body_style 1)
+		(exclude_from_sim no)
+		(in_bom yes)
+		(on_board yes)
+		(in_pos_files yes)
+		(dnp no)
+		(property "Reference" "#PWR0109"
+			(at 67.31 68.58 0)
+			(hide yes)
+			(show_name no)
+			(do_not_autoplace no)
+			(effects
+				(font
+					(size 1.27 1.27)
+				)
+			)
+		)
+		(property "Value" "+3V3_PCIe"
+			(at 74.3712 68.961 90)
+			(show_name no)
+			(do_not_autoplace no)
+			(effects
+				(font
+					(size 1.27 1.27)
+				)
+				(justify left)
+			)
+		)
+		(property "Footprint" ""
+			(at 71.12 68.58 0)
+			(hide yes)
+			(show_name no)
+			(do_not_autoplace no)
+			(effects
+				(font
+					(size 1.27 1.27)
+				)
+			)
+		)
+		(property "Datasheet" ""
+			(at 71.12 68.58 0)
+			(hide yes)
+			(show_name no)
+			(do_not_autoplace no)
+			(effects
+				(font
+					(size 1.27 1.27)
+				)
+			)
+		)
+		(property "Description" ""
+			(at 71.12 68.58 0)
+			(show_name no)
+			(do_not_autoplace no)
+			(effects
+				(font
+					(size 1.27 1.27)
+				)
+			)
+		)
+		(pin "1"
+		)
+		(instances
+			(project "ulx5-PCIe-1x"
+				(path "/9e5cbfd6-8186-4817-919e-acd256336bc8/3b67bf4d-c966-4618-b78c-abe52a948139"
+					(reference "#PWR0109")
+					(unit 1)
+				)

Commit message: Pair switch
Connections:
- net PCIe_RX_N: now also J2.B15 (PETn0)
- net PCIe_RX_P: now also J2.B14 (PETp0)
- net PCIe_TX_N: no longer J2.B15 (PETn0)
- net PCIe_TX_P: no longer J2.B14 (PETp0)
Changed lines of the file:
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@@
 	)
 	(label "PCIe_TX_P"
-		(at 123.19 137.16 180)
+		(at 124.46 143.51 180)
 		(effects
 			(font
@@
 	)
 	(label "PCIe_RX_P"
-		(at 124.46 143.51 180)
+		(at 123.19 137.16 180)
 		(effects
 			(font
@@
 	)
 	(label "PCIe_TX_N"
-		(at 123.19 139.7 180)
+		(at 124.46 146.05 180)
 		(effects
 			(font
@@
 	)
 	(label "PCIe_RX_N"
-		(at 124.46 146.05 180)
+		(at 123.19 139.7 180)
 		(effects
 			(font

Commit message: Fixing diff lines
Connections:
- net CLKREQ#: now reaches J2.B12 (RSVD)
Changed lines of the file:
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@@
+	(wire
+		(pts
+			(xy 120.65 81.28) (xy 125.73 81.28)
+		)
+		(stroke
+			(width 0)
+			(type default)
+		)
+	)
 	(wire
 		(pts
@@
 			)
 			(justify left)
+		)
+	)
+	(hierarchical_label "CLKREQ#"
+		(shape input)
+		(at 120.65 81.28 180)
+		(effects
+			(font
+				(size 1.27 1.27)
+			)
+			(justify right)
 		)
 	)
@@
 			(show_name no)
 			(do_not_autoplace no)
+			(effects
+				(font
+					(size 1.27 1.27)
+				)
+			)
+		)
+		(property "LCSC" ""
+			(at 140.97 48.26 0)
+			(hide yes)
+			(show_name no)
+			(do_not_autoplace no)
