File: lvds.kicad_sch (KiCad schematic)
At the start: 28 parts, among them U4 GateMate-CCGM1A1, Y1 ASE2-25.000MHZ-L-C-T

Commit message: Initial version of 0.2
Connections:
- net +1V2: no longer C49.1, R121.1
- net CLKREQ#: now also U4.V7 (IO_SA_B3); no longer U4.R18 (IO_SB_B1)
- net DEVSLP: now also U4.R7 (IO_SA_A2); no longer U4.U18 (IO_SB_B0)
- net LED1#: now also U4.T6 (IO_SA_B1); no longer U4.M18 (IO_SB_B3)
- net LVDS0_C_N: no longer U4.T9 (IO_SA_B6)
- net LVDS0_C_P: no longer U4.R9 (IO_SA_A6)
- net LVDS0_D0_N: no longer U4.V10 (IO_SA_B8)
- net LVDS0_D0_P: no longer U4.U10 (IO_SA_A8)
- net LVDS0_D1_N: no longer U4.T10 (IO_SA_B7)
- net LVDS0_D1_P: no longer U4.R10 (IO_SA_A7)
- net LVDS0_D2_N: no longer U4.V8 (IO_SA_B5)
- net LVDS0_D2_P: no longer U4.U8 (IO_SA_A5)
- net LVDS0_D3_N: no longer U4.T8 (IO_SA_B4)
- net LVDS0_D3_P: no longer U4.R8 (IO_SA_A4)
- net LVDS1_C_N: no longer U4.T6 (IO_SA_B1)
- net LVDS1_C_P: no longer U4.R6 (IO_SA_A1)
- net LVDS1_D0_N: no longer U4.V7 (IO_SA_B3)
- net LVDS1_D0_P: no longer U4.U7 (IO_SA_A3)
- net LVDS1_D1_N: no longer U4.T7 (IO_SA_B2)
- net LVDS1_D1_P: no longer U4.R7 (IO_SA_A2)
- net LVDS1_D2_N: no longer U4.V5 (IO_SA_B0)
- net LVDS1_D2_P: no longer U4.U5 (IO_SA_A0)
- net PEDET: now also U4.V5 (IO_SA_B0); no longer U4.M17 (IO_SB_A3)
- net PERST#: now also U4.R6 (IO_SA_A1); no longer U4.R17 (IO_SB_A1)
- net PEWAKE#: now also U4.U7 (IO_SA_A3); no longer U4.P17 (IO_SB_A2)
- net SUSCLK: now also U4.T7 (IO_SA_B2); no longer U4.P18 (IO_SB_B2)
- net +1V2_SA renamed +3V3_SA
- new net +3V3: C49.1, R121.1

Commit message: initial version of ULX5-PCIe-1x
Parts:
- removed R129, R130, R131, R132, R135, R136, R50, R51, R54: 150R, Resistor_SMD:R_0402_1005Metric, symbol Device:R_Small
- removed R49, R52, R53, R56, R57, R60: 50R, Resistor_SMD:R_0402_1005Metric, symbol Device:R_Small
- added C259, C260, C261, C262, C263, C264, C265, C266: 220n, Capacitor_SMD:C_0402_1005Metric, symbol Device:C_Small
- added R233, R234, R237, R238, R239, R240, R268, R271, R274: 150R, Resistor_SMD:R_0402_1005Metric, symbol Device:R_Small
- added R67, R69, R70, R72, R73, R75: 50R, Resistor_SMD:R_0402_1005Metric, symbol Device:R_Small
Connections:
- net +1V2: now also C49.1, R121.1
- net +3V3: now also C56.1, R122.2; no longer C49.1, R121.1
- net CAM0_LP_C_N: now also R69.2
- net CAM0_LP_C_P: now also R67.2
- net CAM0_LP_D0_N: now also R72.2
- net CAM0_LP_D0_P: now also R70.2
- net CAM0_LP_D1_N: now also R75.2
- net CAM0_LP_D1_P: now also R73.2
- net CLKREQ#: now also U4.M18 (IO_SB_B3); no longer U4.V7 (IO_SA_B3)
- net DDMI0_HS_CLK_N: now also C266.2
- net DDMI0_HS_CLK_P: now also C265.2
- net DDMI0_HS_TX0_N: now also C260.2
- net DDMI0_HS_TX0_P: now also C259.2
- net DDMI0_HS_TX1_N: now also C262.2
- net DDMI0_HS_TX1_P: now also C261.2
- net DDMI0_HS_TX2_N: now also C264.2
- net DDMI0_HS_TX2_P: now also C263.2
- net DEVSLP: now also U4.P17 (IO_SB_A2); no longer U4.R7 (IO_SA_A2)
- net LED1#: now also U4.R18 (IO_SB_B1); no longer U4.T6 (IO_SA_B1)
- net LVDS0_C_N: now also U4.T9 (IO_SA_B6), R268.2, R69.1
- net LVDS0_C_P: now also U4.R9 (IO_SA_A6), R268.1, R67.1
- net LVDS0_D0_N: now also U4.V10 (IO_SA_B8), R271.2, R72.1
- net LVDS0_D0_P: now also U4.U10 (IO_SA_A8), R271.1, R70.1
- net LVDS0_D1_N: now also U4.T10 (IO_SA_B7), R274.2, R75.1
- net LVDS0_D1_P: now also U4.R10 (IO_SA_A7), R274.1, R73.1
- net LVDS0_D2_N: now also U4.V8 (IO_SA_B5), R233.2
- net LVDS0_D2_P: now also U4.U8 (IO_SA_A5), R233.1
- net LVDS0_D3_N: now also U4.T8 (IO_SA_B4), R234.2
- net LVDS0_D3_P: now also U4.R8 (IO_SA_A4), R234.1
- net LVDS1_C_N: now also U4.T6 (IO_SA_B1), R237.2
- net LVDS1_C_P: now also U4.R6 (IO_SA_A1), R237.1
- net LVDS1_D0_N: now also U4.V7 (IO_SA_B3), R238.2
- net LVDS1_D0_P: now also U4.U7 (IO_SA_A3), R238.1
- net LVDS1_D1_N: now also U4.T7 (IO_SA_B2), R239.2
- net LVDS1_D1_P: now also U4.R7 (IO_SA_A2), R239.1
- net LVDS1_D2_N: now also U4.V5 (IO_SA_B0), R240.2
- net LVDS1_D2_P: now also U4.U5 (IO_SA_A0), R240.1
- net PEDET: now also U4.U18 (IO_SB_B0); no longer U4.V5 (IO_SA_B0)
- net PERST#: now also U4.R17 (IO_SB_A1); no longer U4.R6 (IO_SA_A1)
- net PEWAKE#: now also U4.M17 (IO_SB_A3); no longer U4.U7 (IO_SA_A3)
- net SUSCLK: now also U4.P18 (IO_SB_B2); no longer U4.T7 (IO_SA_B2)
- net VDD_CLK: no longer C56.1, R122.2
- net +1V8_SB renamed +3V3_SB
- net +3V3_SA renamed +1V2_SA
- new net DDMI0_CLK_N: C266.1
- new net DDMI0_CLK_P: C265.1
- new net DDMI0_TX0_N: C260.1
- new net DDMI0_TX0_P: C259.1
- new net DDMI0_TX1_N: C262.1
- new net DDMI0_TX1_P: C261.1
- new net DDMI0_TX2_N: C264.1
- new net DDMI0_TX2_P: C263.1
Other:
- moved on the sheet: C4, Y1

Commit message: Fixing diff lines
Parts:
- added JP303: LVDS-1V2-1V8, Jumper:SolderJumper-3_P1.3mm_Bridged2Bar12_RoundedPad1.0x1.5mm, symbol Jumper:SolderJumper_3_Bridged12
- added LED_P502: LowCur_green, LED_SMD:LED_0603_1608Metric, symbol M-SU-12V-v1r1-eagle-import:LED0603
- added R508: 560R 1%, Resistor_SMD:R_0402_1005Metric, symbol M-SU-12V-v1r1-eagle-import:R0402
Connections:
- net +1V2: now also JP303.1 (A); no longer C49.1, R121.1
- net GND: now also LED_P502.1
- net LED1#: now also R508.2
- net VDD_CLK: now also JP303.3 (B)
- new net: C49.1, JP303.2 (C), R121.1
- new net: LED_P502.2, R508.1
