File: ulx5-PCIe-1x.kicad_sch (KiCad schematic)
At the start: 13 parts

Commit message: Fixing diff lines
Other:
- sheet PCIexpress_connector ports: added CLKREQ#; removed none
- sheet lvds ports: added none; removed LED1#
Changed lines of the file:
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@@
 	(wire
 		(pts
-			(xy 135.89 109.22) (xy 156.21 109.22)
+			(xy 135.89 109.22) (xy 165.1 109.22)
 		)
 		(stroke
@@
 	(wire
 		(pts
-			(xy 135.89 119.38) (xy 156.21 119.38)
+			(xy 90.17 101.6) (xy 100.33 101.6)
 		)
 		(stroke
@@
 		)
 	)
-	(wire
+	(bus
 		(pts
-			(xy 90.17 101.6) (xy 100.33 101.6)
+			(xy 201.93 115.57) (xy 201.93 129.54)
 		)
 		(stroke
@@
 	(bus
 		(pts
-			(xy 201.93 115.57) (xy 201.93 129.54)
+			(xy 90.17 96.52) (xy 104.14 96.52)
 		)
 		(stroke
@@
 		)
 	)
-	(bus
+	(wire
 		(pts
-			(xy 90.17 96.52) (xy 104.14 96.52)
+			(xy 90.17 106.68) (xy 95.25 106.68)
 		)
 		(stroke
@@
 		)
 	)
-	(wire
+	(bus
 		(pts
-			(xy 90.17 106.68) (xy 95.25 106.68)
+			(xy 139.7 134.62) (xy 139.7 153.67)
 		)
 		(stroke
@@
 	(bus
 		(pts
-			(xy 139.7 134.62) (xy 139.7 153.67)
+			(xy 195.58 121.92) (xy 195.58 133.35)
 		)
 		(stroke
@@
 	(bus
 		(pts
-			(xy 195.58 121.92) (xy 195.58 133.35)
+			(xy 139.7 134.62) (xy 165.1 134.62)
 		)
 		(stroke
@@
 		)
 	)
-	(bus
+	(wire
 		(pts
-			(xy 139.7 134.62) (xy 165.1 134.62)
+			(xy 97.79 133.35) (xy 104.14 133.35)
 		)
 		(stroke
@@
 		)
 	)
-	(wire
+	(bus
 		(pts
-			(xy 97.79 133.35) (xy 104.14 133.35)
+			(xy 201.93 129.54) (xy 208.28 129.54)
 		)
 		(stroke
@@
 		)
 	)
-	(bus
+	(wire
 		(pts
-			(xy 201.93 129.54) (xy 208.28 129.54)
+			(xy 135.89 104.14) (xy 165.1 104.14)
 		)
 		(stroke
@@
 	(wire
 		(pts
-			(xy 135.89 104.14) (xy 165.1 104.14)
+			(xy 100.33 101.6) (xy 100.33 130.81)
 		)
 		(stroke
@@
 	(wire
 		(pts
-			(xy 100.33 101.6) (xy 100.33 130.81)
+			(xy 97.79 104.14) (xy 97.79 133.35)
 		)
 		(stroke
@@
 		)
 	)
-	(wire
-		(pts
-			(xy 97.79 104.14) (xy 97.79 133.35)
-		)
-		(stroke
-			(width 0)
-			(type default)
-		)
-	)
 	(label "PEWAKE#"
 		(at 148.59 106.68 180)
-		(effects
-			(font
-				(size 1.27 1.27)
-			)
-			(justify right bottom)
-		)
-	)
-	(label "LED1#"
-		(at 148.59 119.38 180)
 		(effects
 			(font
@@
 			)
 		)
+		(pin "CLKREQ#" input
+			(at 165.1 109.22 180)
+			(effects
+				(font
+					(size 1.27 1.27)
+				)
+				(justify left)
+			)
+		)
 		(instances
 			(project "ulx5-PCIe-1x"
@@
 			(effects
 				(font
-					(size 1.27 1.27)
-				)
-				(justify right)
-			)
-		)
-		(pin "LED1#" output
-			(at 135.89 119.38 0)
-			(effects
-				(font
